File: board/io.kicad_sch (KiCad schematic)
At the start: 9 parts, among them J1 Conn_02x10_Odd_Even, U5 LD1086D2T33TR

Commit message: add title
Other:
- title: (none) -> https://github.com/Lougous/b68k-io
Changed lines of the file:
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@@
 (kicad_sch (version 20211123) (generator eeschema)
   (paper "A4")
+  (title_block
+    (title "https://github.com/Lougous/b68k-io")
+  )
   (junction (at 111.76 184.15) (diameter 0) (color 0 0 0 0)
   )
