File: board/mgr-pic.kicad_sch (KiCad schematic)
At the start: 16 parts, among them J10 Conn_01x06, J12 Conn_01x03, J5 Conn_01x02, U2 PIC18F24K22-xSP-MCU_Microchip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, U3 74LS138

Commit message: add title
Other:
- title: (none) -> https://github.com/Lougous/b68k-io
Changed lines of the file:
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@@
 (kicad_sch (version 20211123) (generator eeschema)
   (paper "A4")
+  (title_block
+    (title "https://github.com/Lougous/b68k-io")
+  )
   (junction (at 140.97 48.26) (diameter 0) (color 0 0 0 0)
   )
