File: board/rs232.kicad_sch (KiCad schematic)
At the start: 7 parts, among them J9 DB9_Male_MountingHoles, U7 MAX232

Commit message: add title
Other:
- title: (none) -> https://github.com/Lougous/b68k-io
Changed lines of the file:
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@@
 (kicad_sch (version 20211123) (generator eeschema)
   (paper "A4")
+  (title_block
+    (title "https://github.com/Lougous/b68k-io")
+  )
   (junction (at 152.4 116.84) (diameter 0) (color 0 0 0 0)
   )
