File: board/rtc.kicad_sch (KiCad schematic)
At the start: 8 parts, among them J6 Conn_01x04, U1 DS1307+, Y1 Crystal

Commit message: add title
Other:
- title: (none) -> https://github.com/Lougous/b68k-io
Changed lines of the file:
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@@
 (kicad_sch (version 20211123) (generator eeschema)
   (paper "A4")
+  (title_block
+    (title "https://github.com/Lougous/b68k-io")
+  )
   (junction (at 134.62 73.66) (diameter 0) (color 0 0 0 0)
   )
