File: board/spi.kicad_sch (KiCad schematic)
At the start: 26 parts, among them J11 Conn_01x08, J2 SD_Card, J3 DB15_Male_MountingHoles, J4 Conn_01x06, J7 SD_Card, J8 Conn_01x06, U4 74LVC244, U6 74LVC244

Commit message: add title
Other:
- title: (none) -> https://github.com/Lougous/b68k-io
Changed lines of the file:
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@@
 (kicad_sch (version 20211123) (generator eeschema)
   (paper "A4")
+  (title_block
+    (title "https://github.com/Lougous/b68k-io")
+  )
   (junction (at 241.3 130.81) (diameter 0) (color 0 0 0 0)
   )
